File: digital-ps.sch (EAGLE design)
At the start: 104 parts, among them CON1 SWD_CON, IC1 3.3V, IC2 7805, IC3 STM32F334K8, IC4 OPA, IC5 MCP14700, Q1 EPC2052, Q2 EPC2052, T1 COMMON_FILTER-SMALL, T2 COMMON_FILTER-SMALL, X1 12MHz

Commit message: GaN
Parts:
- added C42: 470, my_rcl:C-1608-2
- added C43: 10u, my_rcl:C-3225-2
- added R19: 2, my_rcl:R-1608-2
- C19: value 1u -> 10u; device my_rcl:C-1608-2 -> my_rcl:C-3225-2
- C28, C29: value 10u -> 1u; device my_rcl:C-3225-2 -> my_rcl:C-1608-2
- C30: device my_rcl:C-3225-2 -> my_rcl:C-1608-2
- C31: value 0.1u -> 1u; device my_rcl:C-3225-2 -> my_rcl:C-1608-2
- Q1, Q2: device my_ic:NMOS-DFN -> my_ic:NMOS-EPC2055
Connections:
- new net N$9: C42.1, R19.1
- net GND: now also C42.2, C43.2
- net SW: now also R19.2
- net VP: now also C43.1
Other:
- moved on the sheet: C18, C19, C22, C24, C25, C26
